File: Z-.kicad_pcb (KiCad board)
At the start: 4 copper layers, 98 x 98 mm, 142 parts, among them J1 200528-0100, J2 U.FL, J3 U.FL, J5 Conn_01x02, K1 IM11DGR, Q1 NX3008NBKS, Q10 MBT2222ADW1T1, Q11 NX3008NBKS, Q12 MBT2222ADW1T1, Q15 IRFTS9342PBF, Q17 IRFTS9342PBF, Q19 IRFTS9342PBF, Q2 MBT2222ADW1T1, Q20 IRLML2803, Q21 SiRA99DP, Q3 NX3008NBKS, Q4 MBT2222ADW1T1, Q5 NX3008NBKS, Q6 MBT2222ADW1T1, Q7 NX3008NBKS, Q8 MBT2222ADW1T1, Q9 NX3008NBKS, U1 OPT4003DNPRQ1, U2 PCA9633DP2, U4 DRV8235RTER, U5 USBLC6-2P6

Commit message: Added more silkscreen, switched to PMOS instead of mech relay
Parts:
- removed C16: 10uF, Capacitor_SMD:C_1206_3216Metric
- removed D1: PTVS5V0Z1USK, Diode_SMD:Nexperia_DSN1608-2_1.6x0.8mm
- removed K1: IM11DGR, Argus-Miscellaneous:RELAY8_SMTGUL_TEC
- added D8: GREEN, LED_SMD:LED_0603_1608Metric, B.Cu at (144.3, 84.6)
- added F7: 2A, Fuse:Fuse_0603_1608Metric, B.Cu at (156.7, 67.3)
- added Q13: IRLML2803, Package_TO_SOT_SMD:SOT-23, B.Cu at (144.3, 80.8)
- added Q14: SiRA99DP, Argus-Miscellaneous:PowerPAK SO-8, B.Cu at (140.0, 76.1)
- added R68: 2.7k, Resistor_SMD:R_0603_1608Metric, B.Cu at (141.0, 86.1)
- added R69: 10k, Resistor_SMD:R_0603_1608Metric, B.Cu at (133.1, 85.3)
- added R70: 4k7, Resistor_SMD:R_0603_1608Metric, B.Cu at (141.0, 84.6)
- added R73: 10k, Resistor_SMD:R_0603_1608Metric, B.Cu at (145.3, 77.2)
- moved D7 2.09 mm to (136.4, 78.5), turned to -90 degrees
Routing:
- net PERI_3V3: track 84.5 -> 59.2 mm
- net LS_3V3: track 121.3 -> 113.1 mm
- net Net-(Q13-D): track 0.00 -> 4.75 mm
- net Net-(Q13-G): track 0.00 -> 3.50 mm
- net Net-(D8-A): track 0.00 -> 2.32 mm
- net BURN_RELAY_A: track 17.8 -> 16.2 mm
- net GND: track 47.3 -> 47.9 mm, vias 135 -> 130
- added copper zone on B.Cu, net Net-(Q14-S)
Other:
- board text added: "ARGUS"
- board text added: "BATT"
- board text removed: "ARGUS-1"
