File: I2CDevices.kicad_sch (KiCad schematic)
At the start: 37 parts, among them Q20 IRLML2803, Q21 SiRA99DP, U1 OPT4003DNPRQ1, U2 PCA9633DP2, U4 DRV8235RTER

Commit message: push
Connections:
- net BURN_EN1: now also U2.1 (LED0); no longer U2.2 (LED1)
- net BURN_EN2: now also U2.2 (LED1); no longer U2.1 (LED0)
Changed lines of the file:
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@@
 	(global_label "BURN_EN1"
 		(shape bidirectional)
-		(at 36.83 125.73 180)
+		(at 36.83 123.19 180)
 		(effects
 			(font
@@
 		)
 		(property "Intersheetrefs" "${INTERSHEET_REFS}"
-			(at 36.83 125.73 0)
+			(at 36.83 123.19 0)
 			(effects
 				(font
@@
 	(global_label "BURN_EN2"
 		(shape bidirectional)
-		(at 36.83 123.19 180)
+		(at 36.83 125.73 180)
 		(effects
 			(font
@@
 		)
 		(property "Intersheetrefs" "${INTERSHEET_REFS}"
-			(at 36.83 123.19 0)
+			(at 36.83 125.73 0)
 			(effects
 				(font
