File: Z-.kicad_sch (KiCad schematic)
At the start: 27 parts, among them J1 200528-0100, J2 U.FL, J3 U.FL, J5 Conn_01x02, U5 USBLC6-2P6

Commit message: push
Parts:
- removed U5: USBLC6-2P6, Package_TO_SOT_SMD:SOT-666, symbol Power_Protection:USBLC6-2P6
- added U3: USBLC6-2P6, Package_TO_SOT_SMD:SOT-666, symbol Power_Protection:USBLC6-2P6
- AE1, AE2: footprint Argus-Miscellaneous:Antenna Mount -> Argus-Miscellaneous:Antenna Mount v2
Connections:
- net GND: now also U3.2 (GND)
- net MAIN_3V3: now also U3.5 (VBUS)
- net SCL: now also U3.4 (I/O2)
- net SDA: now also U3.6 (I/O1)
- net at J1.1 (Pin_1): now also U3.3 (I/O2)
- net at J1.2 (Pin_2): now also U3.1 (I/O1)
