File: CoilDriver.kicad_sch (KiCad schematic)
At the start: 25 parts, among them Q12 IRLML2803, Q13 SIRA99DP-T1-GE3, U3 DRV8235RTER

Commit message: Stash 2
Parts:
- R50: value TBD -> 2k7
- R51: value TBD -> 1M
Changed lines of the file:
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@@
 			)
 		)
-		(property "Value" "TBD"
+		(property "Value" "2k7"
 			(at 231.14 136.906 0)
 			(effects
@@
 			)
 		)
-		(property "Value" "TBD"
+		(property "Value" "1M"
 			(at 231.14 147.066 0)
 			(effects
